File: esquemáticos/fuente_conmutada_pruebas/fuente_conmutada_pruebas.kicad_sch (KiCad schematic)
At the start: 14 parts, among them Q1 NPN, Q2 N-Channel

Commit message: Fuente acabada?
Parts:
- removed C1: 1000uF, symbol Device:C_Polarized_US
- removed FBR1: KBPC1501T, Diode_THT:Diode_Bridge_Round_D9.8mm, symbol Diode_Bridge:KBPC1501T
- removed M1: ~, symbol Teoría de Circuitos:Motor_DC
- removed Q1: NPN, symbol Simulation_SPICE:NPN
- removed Q2: N-Channel, Package_TO_SOT_SMD:SOT-223-3_TabPin2, symbol Transistor_FET:NDT3055L
- removed RV1: 100k, symbol Device:R_Potentiometer_US
- removed TR1: 11.5:1, symbol Teoría de Circuitos:Transformer
- removed VAC1: 230V, symbol Teoría de Circuitos:AC_source
- added C1: 100n, symbol Device:C
- added Q1: IRLZ24, Package_TO_SOT_THT:TO-220-3_Vertical, symbol Transistor_FET:IRLZ24
- added R6: 100k, symbol Device:R_US
- C2: value 1000uF -> 100n
- R1: value 100k -> 300
- R2: value 100k 1W -> 1k
- R3: value 10k -> 300k
- R4: value 0.03 -> 100k
- R5: value 100k 1W -> 300k
Connections:
- net PWM is gone; now on net VDC: R1.1
- net OSC 2: now reaches R1.2
- net OSC 2: now also R3.1, Q1.2 (D)
- net at R4.1: now also R3.2, C1.1
- net Earth: now reaches C2.2
- net Earth: now also R4.2, C1.2, Q1.3 (S), R6.2
- net GND renamed VDC
- new net: C2.1, R5.2, R6.1
- new net: Q1.1 (G), R2.2
- new net OSC 1: R2.1
Other:
- note removed: "Importante conectar las tierras juntas."
- note removed: "Regulación PWM mediante Arduino (10 bits)."
- note removed: "Shunt"
